File: ergogen/output/pcbs/main.kicad_pcb (KiCad board)
At the start: 2 copper layers, 327.9 x 116.2 mm, 162 parts

Commit message: Updated ergogen config - Added mounting holes - Added board text
Parts:
- removed the _1 at (296.9, -3.55) (x2)
- added ?: , HOLE_M2_TH, F.Cu at (12.0, -19.1)
- added ?: , HOLE_M2_TH, F.Cu at (121.2, 76.2)
- added ?: , HOLE_M2_TH, F.Cu at (251.1, 76.2)
- added ?: , HOLE_M2_TH, F.Cu at (302.9, 57.1)
- added ?: , HOLE_M2_TH, F.Cu at (93.2, -19.1)
- added ?: , HOLE_M2_TH, F.Cu at (174.4, -19.1)
- added ?: , HOLE_M2_TH, F.Cu at (255.7, -19.1)
- added ?: , HOLE_M2_TH, F.Cu at (272.9, 0.00)
- added ?: , HOLE_M2_TH, F.Cu at (17.2, 19.1)
- added ?: , HOLE_M2_TH, F.Cu at (138.9, 28.6)
- added ?: , HOLE_M2_TH, F.Cu at (239.2, 38.1)
- added ?: , HOLE_M2_TH, F.Cu at (28.4, 57.1)
- added _1 (x2): RPi_Pico_SMD_TH, RPi_Pico_SMD_TH, F.Cu at (296.9, -4.05)
Other:
- board text added: "Flatbread v0.1"
Changed lines of the file:
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@@
     )
         (module RPi_Pico_SMD_TH (layer F.Cu)
-        (at 296.9 -3.5500000000000007 0)
+        (at 296.9 -4.050000000000001 0)
         (fp_text reference "_1" (at 0 0) (layer F.SilkS) hide (effects (font (size 1 1) (thickness 0.15))))
         (fp_text value RPi_Pico_SMD_TH (at 0 2.159) (layer F.Fab) (effects (font (size 1 1) (thickness 0.15))))
@@
     )
         (module RPi_Pico_SMD_TH (layer F.Cu)
-        (at 296.9 -3.5500000000000007 0)
+        (at 296.9 -4.050000000000001 0)
         (fp_text reference "_1" (at 0 0) (layer B.SilkS) hide (effects (font (size 1 1) (thickness 0.15))))
         (fp_text value RPi_Pico_SMD_TH (at 0 2.159) (layer F.Fab) (effects (font (size 1 1) (thickness 0.15))))
@@
         (pad 40 smd rect (at 8.89 -24.13 0) (size 3.5 1.7) (drill (offset 0.9 0)) (layers B.Cu B.Mask) (net 111 "VBUS"))
     )
+    (module HOLE_M2_TH (layer F.Cu)
+      (at 12 -19.05 0)
+      (pad "" np_thru_hole circle (at 0 0 90) (size 4.0 4.0) (drill 4.0) (layers *.Cu *.Mask F.SilkS) (clearance 0.3)))
+    (module HOLE_M2_TH (layer F.Cu)
+      (at 93.225 -19.05 0)
+      (pad "" np_thru_hole circle (at 0 0 90) (size 4.0 4.0) (drill 4.0) (layers *.Cu *.Mask F.SilkS) (clearance 0.3)))
+    (module HOLE_M2_TH (layer F.Cu)
+      (at 174.45 -19.05 0)
+      (pad "" np_thru_hole circle (at 0 0 90) (size 4.0 4.0) (drill 4.0) (layers *.Cu *.Mask F.SilkS) (clearance 0.3)))
+    (module HOLE_M2_TH (layer F.Cu)
+      (at 255.675 -19.05 0)
+      (pad "" np_thru_hole circle (at 0 0 90) (size 4.0 4.0) (drill 4.0) (layers *.Cu *.Mask F.SilkS) (clearance 0.3)))
+    (module HOLE_M2_TH (layer F.Cu)
+      (at 272.925 0 0)
+      (pad "" np_thru_hole circle (at 0 0 90) (size 4.0 4.0) (drill 4.0) (layers *.Cu *.Mask F.SilkS) (clearance 0.3)))
+    (module HOLE_M2_TH (layer F.Cu)
+      (at 17.225 19.05 0)
+      (pad "" np_thru_hole circle (at 0 0 90) (size 4.0 4.0) (drill 4.0) (layers *.Cu *.Mask F.SilkS) (clearance 0.3)))
+    (module HOLE_M2_TH (layer F.Cu)
+      (at 138.95 28.55 0)
+      (pad "" np_thru_hole circle (at 0 0 90) (size 4.0 4.0) (drill 4.0) (layers *.Cu *.Mask F.SilkS) (clearance 0.3)))
+    (module HOLE_M2_TH (layer F.Cu)
+      (at 239.2 38.1 0)
+      (pad "" np_thru_hole circle (at 0 0 90) (size 4.0 4.0) (drill 4.0) (layers *.Cu *.Mask F.SilkS) (clearance 0.3)))
+    (module HOLE_M2_TH (layer F.Cu)
+      (at 28.35 57.15 0)
+      (pad "" np_thru_hole circle (at 0 0 90) (size 4.0 4.0) (drill 4.0) (layers *.Cu *.Mask F.SilkS) (clearance 0.3)))
+    (module HOLE_M2_TH (layer F.Cu)
+      (at 121.17499999999998 76.2 0)
+      (pad "" np_thru_hole circle (at 0 0 90) (size 4.0 4.0) (drill 4.0) (layers *.Cu *.Mask F.SilkS) (clearance 0.3)))
+    (module HOLE_M2_TH (layer F.Cu)
+      (at 251.125 76.2 0)
+      (pad "" np_thru_hole circle (at 0 0 90) (size 4.0 4.0) (drill 4.0) (layers *.Cu *.Mask F.SilkS) (clearance 0.3)))
+    (module HOLE_M2_TH (layer F.Cu)
+      (at 302.90000000000003 57.15 0)
+      (pad "" np_thru_hole circle (at 0 0 90) (size 4.0 4.0) (drill 4.0) (layers *.Cu *.Mask F.SilkS) (clearance 0.3)))
+            (gr_text "Flatbread v0.1" (at 156.67499999999998 76.2 0) (layer F.SilkS)
+                (effects (font (size 3 3) (thickness 0.4) ) (justify left))
+            )
   (gr_line (start -11 84.7) (end -11 -27.55) (angle 90) (layer Edge.Cuts) (width 0.15))
 (gr_line (start -9 -29.55) (end 314.9 -29.55) (angle 90) (layer Edge.Cuts) (width 0.15))

Commit message: Case 3D Model - Added mounting points for M2 screws
Parts:
- removed the ? at (272.9, 0.00)
- removed the _1 at (296.9, -4.05) (x2)
- added _1 (x2): RPi_Pico_SMD_TH, RPi_Pico_SMD_TH, F.Cu at (296.9, -4.05)
Changed lines of the file:
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@@
-      (pad "" np_thru_hole circle (at 0 0 90) (size 4.0 4.0) (drill 4.0) (layers *.Cu *.Mask F.SilkS) (clearance 0.3)))
-    (module HOLE_M2_TH (layer F.Cu)
-      (at 272.925 0 0)
       (pad "" np_thru_hole circle (at 0 0 90) (size 4.0 4.0) (drill 4.0) (layers *.Cu *.Mask F.SilkS) (clearance 0.3)))
     (module HOLE_M2_TH (layer F.Cu)

Commit message: Moved mounting holes to make way for stabilizers - Stabilizer slots have been made in the faceplate outline
Parts:
- removed the ? at (239.2, 38.1)
- removed the ? at (28.4, 57.1)
- removed the _1 at (296.9, -4.05) (x2)
- added ?: , HOLE_M2_TH, F.Cu at (224.2, 47.6)
- added ?: , HOLE_M2_TH, F.Cu at (32.7, 65.7)
- added _1 (x2): RPi_Pico_SMD_TH, RPi_Pico_SMD_TH, F.Cu at (296.9, -4.05)
Connections:
- D55 pad 2: backslash_row -> enter_row
- S55 pad 2: backslash_row -> enter_row
Other:
- board text added: "Flatbread v0.2"
- board text removed: "Flatbread v0.1"
